Commit message: Add mapping and urdf for individual robots

File: src/guide_robot/urdf/robot_m.urdf.xacro (robot description, xacro)
@@ -3,5 +3,5 @@
   <xacro:arg name="namespace" default="robot_m" />
   <xacro:include filename="$(find turtlebot3_description)/urdf/common_properties.xacro"/>
-  <xacro:include filename="$(find guide_robot)/urdf/robot.gazebo.xacro"/>
+  <xacro:include filename="$(find guide_robot)/urdf/$(arg namespace).gazebo.xacro"/>
   <xacro:property name="r200_cam_rgb_px" value="0.005"/>
   <xacro:property name="r200_cam_rgb_py" value="0.018"/>

File: src/guide_robot/urdf/robot_s.gazebo.xacro (robot description, xacro)
@@ -105,39 +105,6 @@
     </plugin>
   </gazebo>
-  <gazebo reference="base_scan">
-    <material>Gazebo/FlatBlack</material>
-    <sensor type="ray" name="lds_lfcd_sensor">
-      <pose>0 0 0 0 0 0</pose>
-      <visualize>$(arg laser_visual)</visualize>
-      <update_rate>5</update_rate>
-      <ray>
-        <scan>
-          <horizontal>
-            <samples>360</samples>
-            <resolution>1</resolution>
-            <min_angle>0.0</min_angle>
-            <max_angle>6.28319</max_angle>
-          </horizontal>
-        </scan>
-        <range>
-          <min>0.120</min>
-          <max>3.5</max>
-          <resolution>0.015</resolution>
-        </range>
-        <noise>
-          <type>gaussian</type>
-          <mean>0.0</mean>
-          <stddev>0.01</stddev>
-        </noise>
-      </ray>
-      <plugin name="gazebo_ros_lds_lfcd_controller" filename="libgazebo_ros_laser.so">
-        <robotNamespace>$(arg namespace)</robotNamespace>
-        <topicName>scan</topicName>
-        <frameName>$(arg namespace)/base_scan</frameName>
-      </plugin>
-    </sensor>
-  </gazebo>
   <gazebo reference="$(arg namespace)/camera_rgb_frame">
-    <sensor type="depth" name="realsense_R200">
+    <sensor type="camera" name="realsense_R200">
       <always_on>true</always_on>
       <visualize>$(arg camera_visual)</visualize>
@@ -149,5 +116,4 @@
               <format>R8G8B8</format>
           </image>
-          <depth_camera></depth_camera>
           <clip>
               <near>0.03</near>
@@ -155,28 +121,18 @@
           </clip>
       </camera>
-      <plugin name="camera_controller" filename="libgazebo_ros_openni_kinect.so">
+      <plugin name="camera_controller" filename="libgazebo_ros_camera.so">
         <robotNamespace>$(arg namespace)</robotNamespace>
-        <baseline>0.2</baseline>
         <alwaysOn>true</alwaysOn>
         <updateRate>30.0</updateRate>
         <cameraName>camera</cameraName>
+        <imageTopicName>rgb/image_raw</imageTopicName>
+        <cameraInfoTopicName>rgb/camera_info</cameraInfoTopicName>
         <frameName>$(arg namespace)/camera_rgb_optical_frame</frameName>
-        <imageTopicName>rgb/image_raw</imageTopicName>
-        <depthImageTopicName>depth/image_raw</depthImageTopicName>
-        <pointCloudTopicName>depth/points</pointCloudTopicName>
-        <cameraInfoTopicName>rgb/camera_info</cameraInfoTopicName>
-        <depthImageCameraInfoTopicName>depth/camera_info</depthImageCameraInfoTopicName>
-        <pointCloudCutoff>0.4</pointCloudCutoff>
-            <hackBaseline>0.07</hackBaseline>
-            <distortionK1>0.0</distortionK1>
-            <distortionK2>0.0</distortionK2>
-            <distortionK3>0.0</distortionK3>
-            <distortionT1>0.0</distortionT1>
-            <distortionT2>0.0</distortionT2>
-        <CxPrime>0.0</CxPrime>
-        <Cx>0.0</Cx>
-        <Cy>0.0</Cy>
-        <focalLength>0</focalLength>
-        <hackBaseline>0</hackBaseline>
+        <hackBaseline>0.07</hackBaseline>
+        <distortionK1>0.0</distortionK1>
+        <distortionK2>0.0</distortionK2>
+        <distortionK3>0.0</distortionK3>
+        <distortionT1>0.0</distortionT1>
+        <distortionT2>0.0</distortionT2>
       </plugin>
     </sensor>

Commit message: Add maps for hospital

File: src/guide_robot/urdf/robot_m.urdf.xacro (robot description, xacro)
@@ -14,4 +14,9 @@
     <origin xyz="0 0 0.010" rpy="0 0 0"/>
   </joint>
+  <!-- adding apriltag -->
+  <joint name="$(arg namespace)/aprilTag" type="fixed">
+      <parent link="$(arg namespace)/base_footprint"/>
+      <origin xyz="0 0 0.010" rpy="0 1.57 0"/>
+   </joint>
   <link name="$(arg namespace)/base_link">
     <visual>
