Commit message: .

File: src/guide_robot/urdf/robot_m.gazebo.xacro (robot description, xacro)
@@ -8,4 +8,8 @@
     <material>Gazebo/DarkGrey</material>
   </gazebo>
+  <!-- Add april tag -->
+  <!-- <gazebo reference="$(arg namespace)/aprilTag">
+    <material>Gazebo/FlatBlack</material>
+  </gazebo> -->
   <gazebo reference="$(arg namespace)/wheel_left_link">
     <mu1>0.1</mu1>

File: src/guide_robot/urdf/robot_m.urdf.xacro (robot description, xacro)
@@ -15,6 +15,15 @@
   </joint>
   <!-- adding apriltag -->
-  <joint name="$(arg namespace)/aprilTag" type="fixed">
-      <parent link="$(arg namespace)/base_footprint"/>
+  <link name="$(arg namespace)/aprilTag"/>
+    <visual>
+      <origin xyz="0 0 0" rpy="0 1.57 0"/>
+      <geometry>
+        <mesh filename="model://tag36h11img-008_out/meshes/tag36h11img-008_out.dae" scale="0.6 0.6 0.6"/>
+      </geometry>
+      <material name="dark"/>
+    </visual>
+  <joint name="$(arg namespace)/aprilTagJoint" type="fixed">
+      <parent link="$(arg namespace)/base_link"/>
+      <child link="$(arg namespace)/aprilTag" />
       <origin xyz="0 0 0.010" rpy="0 1.57 0"/>
    </joint>

Commit message: Get tag detections and slave follower working

File: src/guide_robot/urdf/robot_m.gazebo.xacro (robot description, xacro)
@@ -165,5 +165,5 @@
         <updateRate>30.0</updateRate>
         <cameraName>camera</cameraName>
-        <frameName>$(arg namespace)/camera_rgb_optical_frame</frameName>
+        <frameName>camera_rgb_optical_frame</frameName>
         <imageTopicName>rgb/image_raw</imageTopicName>
         <depthImageTopicName>depth/image_raw</depthImageTopicName>

File: src/guide_robot/urdf/robot_m.urdf.xacro (robot description, xacro)
@@ -15,17 +15,18 @@
   </joint>
   <!-- adding apriltag -->
-  <link name="$(arg namespace)/aprilTag"/>
+  <link name="$(arg namespace)/aprilTag">
     <visual>
       <origin xyz="0 0 0" rpy="0 1.57 0"/>
       <geometry>
-        <mesh filename="model://tag36h11img-008_out/meshes/tag36h11img-008_out.dae" scale="0.6 0.6 0.6"/>
-      </geometry>
-      <material name="dark"/>
-    </visual>
+        <mesh filename="package://guide_robot/meshes/tag36h11img-008_out.dae" scale="0.6 0.6 0.6"/>
+      </geometry>
+      <material name="dark"/>
+    </visual>
+  </link>
   <joint name="$(arg namespace)/aprilTagJoint" type="fixed">
       <parent link="$(arg namespace)/base_link"/>
       <child link="$(arg namespace)/aprilTag" />
-      <origin xyz="0 0 0.010" rpy="0 1.57 0"/>
-   </joint>
+      <origin xyz="0 0 0.410" rpy="0 1.57 0"/>
+  </joint>
   <link name="$(arg namespace)/base_link">
     <visual>

File: src/guide_robot/urdf/robot_s.gazebo.xacro (robot description, xacro)
@@ -128,5 +128,5 @@
         <imageTopicName>rgb/image_raw</imageTopicName>
         <cameraInfoTopicName>rgb/camera_info</cameraInfoTopicName>
-        <frameName>$(arg namespace)/camera_rgb_optical_frame</frameName>
+        <frameName>camera_rgb_optical_frame</frameName>
         <hackBaseline>0.07</hackBaseline>
         <distortionK1>0.0</distortionK1>
